Commit message: adds gazebo integration

File: ros/src/qcar/urdf/qcar_model.xacro (robot description, xacro)
@@ -2,5 +2,5 @@
 <robot name="QCar" xmlns:xacro="http://www.ros.org/wiki/xacro">
   <xacro:include filename="$(find qcar)/urdf/materials.xacro" />
-  <!-- <xacro:include filename="$(find qcar)/urdf/macros.xacro" /> -->
+  <xacro:include filename="$(find realsense2_description)/urdf/_d435.urdf.xacro" />
   <link name="base">
         <visual>
@@ -317,3 +317,6 @@
         </actuator>
     </transmission>
+    <xacro:sensor_d435 name="camera" topics_ns="camera" parent="camera_rgb" publish_pointcloud="true">
+        <origin xyz="0 0 0" rpy="0 0 0" />
+    </xacro:sensor_d435>
   </robot>

Commit message: update with controller

File: ros/src/qcar/urdf/qcar_model.xacro (robot description, xacro)
@@ -122,5 +122,6 @@
             <origin rpy="0 0 0" xyz="0 0 0"/>
             <geometry>
-                <mesh filename="package://qcar/meshes/QCarWheel.stl" scale="0.001 0.001 0.001"/>
+                <!-- <mesh filename="package://qcar/meshes/QCarWheel.stl" scale="0.001 0.001 0.001"/> -->
+                <cylinder length="0.25" radius="0.3" />
             </geometry>
         </collision>
@@ -148,5 +149,6 @@
             <origin rpy="0 0 0" xyz="0 0 0"/>
             <geometry>
-                <mesh filename="package://qcar/meshes/QCarWheel.stl" scale="0.001 0.001 0.001"/>
+                <!-- <mesh filename="package://qcar/meshes/QCarWheel.stl" scale="0.001 0.001 0.001"/> -->
+                <cylinder length="0.25" radius="0.3" />
             </geometry>
         </collision>
@@ -174,5 +176,6 @@
             <origin rpy="0 0 0" xyz="0 0 0"/>
             <geometry>
-                <mesh filename="package://qcar/meshes/QCarWheel.stl" scale="0.001 0.001 0.001"/>
+                <!-- <mesh filename="package://qcar/meshes/QCarWheel.stl" scale="0.001 0.001 0.001"/> -->
+                <cylinder length="0.25" radius="0.3" />
             </geometry>
         </collision>
@@ -200,5 +203,6 @@
             <origin rpy="0 0 0" xyz="0 0 0"/>
             <geometry>
-                <mesh filename="package://qcar/meshes/QCarWheel.stl" scale="0.001 0.001 0.001"/>
+                <!-- <mesh filename="package://qcar/meshes/QCarWheel.stl" scale="0.001 0.001 0.001"/> -->
+                <cylinder length="0.25" radius="0.3" />
             </geometry>
         </collision>
@@ -284,5 +288,5 @@
         <type>>transmission_interface/SimpleTransmission</type>
         <joint name="hubfl_wheelfl_joint">
-            <hardwareInterface>hardware_interface/EffortJointInterface</hardwareInterface>
+            <hardwareInterface>hardware_interface/PositionJointInterface</hardwareInterface>
         </joint>
         <actuator name="hubfl_wheelfl_motor">
@@ -293,5 +297,5 @@
         <type>>transmission_interface/SimpleTransmission</type>
         <joint name="hubfr_wheelfr_joint">
-            <hardwareInterface>hardware_interface/EffortJointInterface</hardwareInterface>
+            <hardwareInterface>hardware_interface/PositionJointInterface</hardwareInterface>
         </joint>
         <actuator name="hubfr_wheelfr_motor">
@@ -302,5 +306,5 @@
         <type>>transmission_interface/SimpleTransmission</type>
         <joint name="base_wheelrl_joint">
-            <hardwareInterface>hardware_interface/EffortJointInterface</hardwareInterface>
+            <hardwareInterface>hardware_interface/VelocityJointInterface</hardwareInterface>
         </joint>
         <actuator name="base_wheelrl_motor">
@@ -311,5 +315,5 @@
         <type>>transmission_interface/SimpleTransmission</type>
         <joint name="base_wheelrr_joint">
-            <hardwareInterface>hardware_interface/EffortJointInterface</hardwareInterface>
+            <hardwareInterface>hardware_interface/VelocityJointInterface</hardwareInterface>
         </joint>
         <actuator name="base_wheelrr_motor">
@@ -320,3 +324,9 @@
         <origin xyz="0 0 0" rpy="0 0 0" />
     </xacro:sensor_d435>
+<!-- Ros Control plugin-->
+    <gazebo>
+        <plugin name="gazebo_ros_control" filename="libgazebo_ros_control.so">
+        <robotNamespace>/</robotNamespace>
+        </plugin>
+    </gazebo>
   </robot>
