Commit message: woooooooooooooooooooooooooo

File: ros/src/qcar_gazebo/urdf/qcar_model.xacro (robot description, xacro)
@@ -1,5 +1,5 @@
 <?xml version='1.0'?>
 <robot name="QCar" xmlns:xacro="http://www.ros.org/wiki/xacro">
-  <xacro:include filename="$(find qcar)/urdf/materials.xacro" />
+  <xacro:include filename="$(find qcar_gazebo)/urdf/materials.xacro" />
   <xacro:include filename="$(find realsense2_description)/urdf/_d435.urdf.xacro" />
   <link name="base">
@@ -7,5 +7,5 @@
             <origin rpy="0 0 0" xyz="0 0 0"/>
             <geometry>
-                <mesh filename="package://qcar/meshes/QCarBody.stl" scale="0.001 0.001 0.001"/>
+                <mesh filename="package://qcar_gazebo/meshes/QCarBody.stl" scale="0.001 0.001 0.001"/>
             </geometry>
             <material name="white"/>
@@ -14,5 +14,5 @@
             <origin rpy="0 0 0" xyz="0 0 0"/>
             <geometry>
-                <mesh filename="package://qcar/meshes/QCarBody.stl" scale="0.001 0.001 0.001"/>
+                <mesh filename="package://qcar_gazebo/meshes/QCarBody.stl" scale="0.001 0.001 0.001"/>
             </geometry>
         </collision>
@@ -33,5 +33,5 @@
             <origin rpy="0 0 0" xyz="0 0 0"/>
             <geometry>
-                <mesh filename="package://qcar/meshes/QCarLidar.stl" scale="0.001 0.001 0.001"/>
+                <mesh filename="package://qcar_gazebo/meshes/QCarLidar.stl" scale="0.001 0.001 0.001"/>
             </geometry>
             <material name="blue"/>
@@ -40,5 +40,5 @@
             <origin rpy="0 0 0" xyz="0 0 0"/>
             <geometry>
-                <mesh filename="package://qcar/meshes/QCarLidar.stl" scale="0.001 0.001 0.001"/>
+                <mesh filename="package://qcar_gazebo/meshes/QCarLidar.stl" scale="0.001 0.001 0.001"/>
             </geometry>
         </collision>
@@ -61,5 +61,5 @@
             <origin rpy="0 0 0" xyz="0 0 0"/>
             <geometry>
-                <mesh filename="package://qcar/meshes/QCarSteeringHubL.stl" scale="0.001 0.001 0.001"/>
+                <mesh filename="package://qcar_gazebo/meshes/QCarSteeringHubL.stl" scale="0.001 0.001 0.001"/>
             </geometry>
             <material name="orange"/>
@@ -68,5 +68,5 @@
             <origin rpy="0 0 0" xyz="0 0 0"/>
             <geometry>
-                <mesh filename="package://qcar/meshes/QCarSteeringHubL.stl" scale="0.001 0.001 0.001"/>
+                <mesh filename="package://qcar_gazebo/meshes/QCarSteeringHubL.stl" scale="0.001 0.001 0.001"/>
             </geometry>
         </collision>
@@ -89,5 +89,5 @@
             <origin rpy="0 0 0" xyz="0 0 0"/>
             <geometry>
-                <mesh filename="package://qcar/meshes/QCarSteeringHubR.stl" scale="0.001 0.001 0.001"/>
+                <mesh filename="package://qcar_gazebo/meshes/QCarSteeringHubR.stl" scale="0.001 0.001 0.001"/>
             </geometry>
             <material name="orange"/>
@@ -96,5 +96,5 @@
             <origin rpy="0 0 0" xyz="0 0 0"/>
             <geometry>
-                <mesh filename="package://qcar/meshes/QCarSteeringHubR.stl" scale="0.001 0.001 0.001"/>
+                <mesh filename="package://qcar_gazebo/meshes/QCarSteeringHubR.stl" scale="0.001 0.001 0.001"/>
             </geometry>
         </collision>
@@ -115,5 +115,5 @@
             <origin rpy="0 0 0" xyz="0 0 0"/>
             <geometry>
-                <mesh filename="package://qcar/meshes/QCarWheel.stl" scale="0.001 0.001 0.001"/>
+                <mesh filename="package://qcar_gazebo/meshes/QCarWheel.stl" scale="0.001 0.001 0.001"/>
             </geometry>
             <material name="red"/>
@@ -122,6 +122,5 @@
             <origin rpy="0 0 0" xyz="0 0 0"/>
             <geometry>
-                <!-- <mesh filename="package://qcar/meshes/QCarWheel.stl" scale="0.001 0.001 0.001"/> -->
-                <cylinder length="0.25" radius="0.3" />
+                <mesh filename="package://qcar_gazebo/meshes/QCarWheel.stl" scale="0.001 0.001 0.001"/>
             </geometry>
         </collision>
@@ -142,5 +141,5 @@
             <origin rpy="0 0 0" xyz="0 0 0"/>
             <geometry>
-                <mesh filename="package://qcar/meshes/QCarWheel.stl" scale="0.001 0.001 0.001"/>
+                <mesh filename="package://qcar_gazebo/meshes/QCarWheel.stl" scale="0.001 0.001 0.001"/>
             </geometry>
             <material name="orange"/>
@@ -149,6 +148,5 @@
             <origin rpy="0 0 0" xyz="0 0 0"/>
             <geometry>
-                <!-- <mesh filename="package://qcar/meshes/QCarWheel.stl" scale="0.001 0.001 0.001"/> -->
-                <cylinder length="0.25" radius="0.3" />
+                <mesh filename="package://qcar_gazebo/meshes/QCarWheel.stl" scale="0.001 0.001 0.001"/>
             </geometry>
         </collision>
@@ -169,5 +167,5 @@
             <origin rpy="0 0 0" xyz="0 0 0"/>
             <geometry>
-                <mesh filename="package://qcar/meshes/QCarWheel.stl" scale="0.001 0.001 0.001"/>
+                <mesh filename="package://qcar_gazebo/meshes/QCarWheel.stl" scale="0.001 0.001 0.001"/>
             </geometry>
             <material name="orange"/>
@@ -176,6 +174,5 @@
             <origin rpy="0 0 0" xyz="0 0 0"/>
             <geometry>
-                <!-- <mesh filename="package://qcar/meshes/QCarWheel.stl" scale="0.001 0.001 0.001"/> -->
-                <cylinder length="0.25" radius="0.3" />
+                <mesh filename="package://qcar_gazebo/meshes/QCarWheel.stl" scale="0.001 0.001 0.001"/>
             </geometry>
         </collision>
@@ -196,5 +193,5 @@
             <origin rpy="0 0 0" xyz="0 0 0"/>
             <geometry>
-                <mesh filename="package://qcar/meshes/QCarWheel.stl" scale="0.001 0.001 0.001"/>
+                <mesh filename="package://qcar_gazebo/meshes/QCarWheel.stl" scale="0.001 0.001 0.001"/>
             </geometry>
             <material name="red"/>
@@ -203,6 +200,5 @@
             <origin rpy="0 0 0" xyz="0 0 0"/>
             <geometry>
-                <!-- <mesh filename="package://qcar/meshes/QCarWheel.stl" scale="0.001 0.001 0.001"/> -->
-                <cylinder length="0.25" radius="0.3" />
+                <mesh filename="package://qcar_gazebo/meshes/QCarWheel.stl" scale="0.001 0.001 0.001"/>
             </geometry>
         </collision>
@@ -270,32 +266,32 @@
         <type>>transmission_interface/SimpleTransmission</type>
         <joint name="base_hubfl_joint">
+            <hardwareInterface>hardware_interface/PositionJointInterface</hardwareInterface>
+        </joint>
+        <actuator name="base_hubfl_motor">
+            <mechanicalReduction>1</mechanicalReduction>
+        </actuator>
+    </transmission>
+    <transmission name="base_hubfr_tran">
+        <type>>transmission_interface/SimpleTransmission</type>
+        <joint name="base_hubfr_joint">
+            <hardwareInterface>hardware_interface/PositionJointInterface</hardwareInterface>
+        </joint>
+        <actuator name="base_hubfr_motor">
+            <mechanicalReduction>1</mechanicalReduction>
+        </actuator>
+    </transmission>
+    <transmission name="hubfl_wheelfl_tran">
+        <type>>transmission_interface/SimpleTransmission</type>
+        <joint name="hubfl_wheelfl_joint">
             <hardwareInterface>hardware_interface/EffortJointInterface</hardwareInterface>
         </joint>
-        <actuator name="base_hubfl_motor">
-            <mechanicalReduction>1</mechanicalReduction>
-        </actuator>
-    </transmission>
-    <transmission name="base_hubfr_tran">
-        <type>>transmission_interface/SimpleTransmission</type>
-        <joint name="base_hubfr_joint">
+        <actuator name="hubfl_wheelfl_motor">
+            <mechanicalReduction>1</mechanicalReduction>
+        </actuator>
+    </transmission>
+    <transmission name="hubfr_wheelfr_tran">
+        <type>>transmission_interface/SimpleTransmission</type>
+        <joint name="hubfr_wheelfr_joint">
             <hardwareInterface>hardware_interface/EffortJointInterface</hardwareInterface>
-        </joint>
-        <actuator name="base_hubfr_motor">
-            <mechanicalReduction>1</mechanicalReduction>
-        </actuator>
-    </transmission>
-    <transmission name="hubfl_wheelfl_tran">
-        <type>>transmission_interface/SimpleTransmission</type>
-        <joint name="hubfl_wheelfl_joint">
-            <hardwareInterface>hardware_interface/PositionJointInterface</hardwareInterface>
-        </joint>
-        <actuator name="hubfl_wheelfl_motor">
-            <mechanicalReduction>1</mechanicalReduction>
-        </actuator>
-    </transmission>
-    <transmission name="hubfr_wheelfr_tran">
-        <type>>transmission_interface/SimpleTransmission</type>
-        <joint name="hubfr_wheelfr_joint">
-            <hardwareInterface>hardware_interface/PositionJointInterface</hardwareInterface>
         </joint>
         <actuator name="hubfr_wheelfr_motor">
@@ -321,11 +317,10 @@
         </actuator>
     </transmission>
-    <xacro:sensor_d435 name="camera" topics_ns="camera" parent="camera_rgb" publish_pointcloud="true">
+    <xacro:sensor_d435 name="camera" topics_ns="camera" parent="camera_rgb">
         <origin xyz="0 0 0" rpy="0 0 0" />
     </xacro:sensor_d435>
-<!-- Ros Control plugin-->
     <gazebo>
         <plugin name="gazebo_ros_control" filename="libgazebo_ros_control.so">
-        <robotNamespace>/</robotNamespace>
+        <robotNamespace>/qcar</robotNamespace>
         </plugin>
     </gazebo>

Commit message: adds gazebo integration (#4)

File: ros/src/qcar_gazebo/urdf/qcar_model.xacro (robot description, xacro)
@@ -1,11 +1,11 @@
 <?xml version='1.0'?>
 <robot name="QCar" xmlns:xacro="http://www.ros.org/wiki/xacro">
-  <xacro:include filename="$(find qcar)/urdf/materials.xacro" />
-  <!-- <xacro:include filename="$(find qcar)/urdf/macros.xacro" /> -->
+  <xacro:include filename="$(find qcar_gazebo)/urdf/materials.xacro" />
+  <xacro:include filename="$(find realsense2_description)/urdf/_d435.urdf.xacro" />
   <link name="base">
         <visual>
             <origin rpy="0 0 0" xyz="0 0 0"/>
             <geometry>
-                <mesh filename="package://qcar/meshes/QCarBody.stl" scale="0.001 0.001 0.001"/>
+                <mesh filename="package://qcar_gazebo/meshes/QCarBody.stl" scale="0.001 0.001 0.001"/>
             </geometry>
             <material name="white"/>
@@ -14,5 +14,5 @@
             <origin rpy="0 0 0" xyz="0 0 0"/>
             <geometry>
-                <mesh filename="package://qcar/meshes/QCarBody.stl" scale="0.001 0.001 0.001"/>
+                <mesh filename="package://qcar_gazebo/meshes/QCarBody.stl" scale="0.001 0.001 0.001"/>
             </geometry>
         </collision>
@@ -33,5 +33,5 @@
             <origin rpy="0 0 0" xyz="0 0 0"/>
             <geometry>
-                <mesh filename="package://qcar/meshes/QCarLidar.stl" scale="0.001 0.001 0.001"/>
+                <mesh filename="package://qcar_gazebo/meshes/QCarLidar.stl" scale="0.001 0.001 0.001"/>
             </geometry>
             <material name="blue"/>
@@ -40,5 +40,5 @@
             <origin rpy="0 0 0" xyz="0 0 0"/>
             <geometry>
-                <mesh filename="package://qcar/meshes/QCarLidar.stl" scale="0.001 0.001 0.001"/>
+                <mesh filename="package://qcar_gazebo/meshes/QCarLidar.stl" scale="0.001 0.001 0.001"/>
             </geometry>
         </collision>
@@ -61,5 +61,5 @@
             <origin rpy="0 0 0" xyz="0 0 0"/>
             <geometry>
-                <mesh filename="package://qcar/meshes/QCarSteeringHubL.stl" scale="0.001 0.001 0.001"/>
+                <mesh filename="package://qcar_gazebo/meshes/QCarSteeringHubL.stl" scale="0.001 0.001 0.001"/>
             </geometry>
             <material name="orange"/>
@@ -68,5 +68,5 @@
             <origin rpy="0 0 0" xyz="0 0 0"/>
             <geometry>
-                <mesh filename="package://qcar/meshes/QCarSteeringHubL.stl" scale="0.001 0.001 0.001"/>
+                <mesh filename="package://qcar_gazebo/meshes/QCarSteeringHubL.stl" scale="0.001 0.001 0.001"/>
             </geometry>
         </collision>
@@ -89,5 +89,5 @@
             <origin rpy="0 0 0" xyz="0 0 0"/>
             <geometry>
-                <mesh filename="package://qcar/meshes/QCarSteeringHubR.stl" scale="0.001 0.001 0.001"/>
+                <mesh filename="package://qcar_gazebo/meshes/QCarSteeringHubR.stl" scale="0.001 0.001 0.001"/>
             </geometry>
             <material name="orange"/>
@@ -96,5 +96,5 @@
             <origin rpy="0 0 0" xyz="0 0 0"/>
             <geometry>
-                <mesh filename="package://qcar/meshes/QCarSteeringHubR.stl" scale="0.001 0.001 0.001"/>
+                <mesh filename="package://qcar_gazebo/meshes/QCarSteeringHubR.stl" scale="0.001 0.001 0.001"/>
             </geometry>
         </collision>
@@ -115,5 +115,5 @@
             <origin rpy="0 0 0" xyz="0 0 0"/>
             <geometry>
-                <mesh filename="package://qcar/meshes/QCarWheel.stl" scale="0.001 0.001 0.001"/>
+                <mesh filename="package://qcar_gazebo/meshes/QCarWheel.stl" scale="0.001 0.001 0.001"/>
             </geometry>
             <material name="red"/>
@@ -122,5 +122,5 @@
             <origin rpy="0 0 0" xyz="0 0 0"/>
             <geometry>
-                <mesh filename="package://qcar/meshes/QCarWheel.stl" scale="0.001 0.001 0.001"/>
+                <mesh filename="package://qcar_gazebo/meshes/QCarWheel.stl" scale="0.001 0.001 0.001"/>
             </geometry>
         </collision>
@@ -141,5 +141,5 @@
             <origin rpy="0 0 0" xyz="0 0 0"/>
             <geometry>
-                <mesh filename="package://qcar/meshes/QCarWheel.stl" scale="0.001 0.001 0.001"/>
+                <mesh filename="package://qcar_gazebo/meshes/QCarWheel.stl" scale="0.001 0.001 0.001"/>
             </geometry>
             <material name="orange"/>
@@ -148,5 +148,5 @@
             <origin rpy="0 0 0" xyz="0 0 0"/>
             <geometry>
-                <mesh filename="package://qcar/meshes/QCarWheel.stl" scale="0.001 0.001 0.001"/>
+                <mesh filename="package://qcar_gazebo/meshes/QCarWheel.stl" scale="0.001 0.001 0.001"/>
             </geometry>
         </collision>
@@ -167,5 +167,5 @@
             <origin rpy="0 0 0" xyz="0 0 0"/>
             <geometry>
-                <mesh filename="package://qcar/meshes/QCarWheel.stl" scale="0.001 0.001 0.001"/>
+                <mesh filename="package://qcar_gazebo/meshes/QCarWheel.stl" scale="0.001 0.001 0.001"/>
             </geometry>
             <material name="orange"/>
@@ -174,5 +174,5 @@
             <origin rpy="0 0 0" xyz="0 0 0"/>
             <geometry>
-                <mesh filename="package://qcar/meshes/QCarWheel.stl" scale="0.001 0.001 0.001"/>
+                <mesh filename="package://qcar_gazebo/meshes/QCarWheel.stl" scale="0.001 0.001 0.001"/>
             </geometry>
         </collision>
@@ -193,5 +193,5 @@
             <origin rpy="0 0 0" xyz="0 0 0"/>
             <geometry>
-                <mesh filename="package://qcar/meshes/QCarWheel.stl" scale="0.001 0.001 0.001"/>
+                <mesh filename="package://qcar_gazebo/meshes/QCarWheel.stl" scale="0.001 0.001 0.001"/>
             </geometry>
             <material name="red"/>
@@ -200,5 +200,5 @@
             <origin rpy="0 0 0" xyz="0 0 0"/>
             <geometry>
-                <mesh filename="package://qcar/meshes/QCarWheel.stl" scale="0.001 0.001 0.001"/>
+                <mesh filename="package://qcar_gazebo/meshes/QCarWheel.stl" scale="0.001 0.001 0.001"/>
             </geometry>
         </collision>
@@ -266,5 +266,5 @@
         <type>>transmission_interface/SimpleTransmission</type>
         <joint name="base_hubfl_joint">
-            <hardwareInterface>hardware_interface/EffortJointInterface</hardwareInterface>
+            <hardwareInterface>hardware_interface/PositionJointInterface</hardwareInterface>
         </joint>
         <actuator name="base_hubfl_motor">
@@ -275,5 +275,5 @@
         <type>>transmission_interface/SimpleTransmission</type>
         <joint name="base_hubfr_joint">
-            <hardwareInterface>hardware_interface/EffortJointInterface</hardwareInterface>
+            <hardwareInterface>hardware_interface/PositionJointInterface</hardwareInterface>
         </joint>
         <actuator name="base_hubfr_motor">
@@ -302,5 +302,5 @@
         <type>>transmission_interface/SimpleTransmission</type>
         <joint name="base_wheelrl_joint">
-            <hardwareInterface>hardware_interface/EffortJointInterface</hardwareInterface>
+            <hardwareInterface>hardware_interface/VelocityJointInterface</hardwareInterface>
         </joint>
         <actuator name="base_wheelrl_motor">
@@ -311,5 +311,5 @@
         <type>>transmission_interface/SimpleTransmission</type>
         <joint name="base_wheelrr_joint">
-            <hardwareInterface>hardware_interface/EffortJointInterface</hardwareInterface>
+            <hardwareInterface>hardware_interface/VelocityJointInterface</hardwareInterface>
         </joint>
         <actuator name="base_wheelrr_motor">
@@ -317,3 +317,11 @@
         </actuator>
     </transmission>
+    <xacro:sensor_d435 name="camera" topics_ns="camera" parent="camera_rgb">
+        <origin xyz="0 0 0" rpy="0 0 0" />
+    </xacro:sensor_d435>
+    <gazebo>
+        <plugin name="gazebo_ros_control" filename="libgazebo_ros_control.so">
+        <robotNamespace>/qcar</robotNamespace>
+        </plugin>
+    </gazebo>
   </robot>
