Commit message: Adjusted gazebo worlds touse dynamic file paths so they work on different PCs

File: ros/src/qcar_gazebo/urdf/qcar_model.xacro (robot description, xacro)
@@ -7,5 +7,5 @@
             <origin rpy="0 0 0" xyz="0 0 0"/>
             <geometry>
-                <mesh filename="package://qcar_gazebo/meshes/QCarBody.stl" scale="0.001 0.001 0.001"/>
+                <mesh filename="package://qcar_gazebo/models/qcar/QCarBody.stl" scale="0.001 0.001 0.001"/>
             </geometry>
             <material name="white"/>
@@ -14,5 +14,5 @@
             <origin rpy="0 0 0" xyz="0 0 0"/>
             <geometry>
-                <mesh filename="package://qcar_gazebo/meshes/QCarBody.stl" scale="0.001 0.001 0.001"/>
+                <mesh filename="package://qcar_gazebo/models/qcar/QCarBody.stl" scale="0.001 0.001 0.001"/>
             </geometry>
         </collision>
@@ -33,5 +33,5 @@
             <origin rpy="0 0 0" xyz="0 0 0"/>
             <geometry>
-                <mesh filename="package://qcar_gazebo/meshes/QCarLidar.stl" scale="0.001 0.001 0.001"/>
+                <mesh filename="package://qcar_gazebo/models/qcar/QCarLidar.stl" scale="0.001 0.001 0.001"/>
             </geometry>
             <material name="blue"/>
@@ -40,5 +40,5 @@
             <origin rpy="0 0 0" xyz="0 0 0"/>
             <geometry>
-                <mesh filename="package://qcar_gazebo/meshes/QCarLidar.stl" scale="0.001 0.001 0.001"/>
+                <mesh filename="package://qcar_gazebo/models/qcar/QCarLidar.stl" scale="0.001 0.001 0.001"/>
             </geometry>
         </collision>
@@ -61,5 +61,5 @@
             <origin rpy="0 0 0" xyz="0 0 0"/>
             <geometry>
-                <mesh filename="package://qcar_gazebo/meshes/QCarSteeringHubL.stl" scale="0.001 0.001 0.001"/>
+                <mesh filename="package://qcar_gazebo/models/qcar/QCarSteeringHubL.stl" scale="0.001 0.001 0.001"/>
             </geometry>
             <material name="orange"/>
@@ -68,5 +68,5 @@
             <origin rpy="0 0 0" xyz="0 0 0"/>
             <geometry>
-                <mesh filename="package://qcar_gazebo/meshes/QCarSteeringHubL.stl" scale="0.001 0.001 0.001"/>
+                <mesh filename="package://qcar_gazebo/models/qcar/QCarSteeringHubL.stl" scale="0.001 0.001 0.001"/>
             </geometry>
         </collision>
@@ -89,5 +89,5 @@
             <origin rpy="0 0 0" xyz="0 0 0"/>
             <geometry>
-                <mesh filename="package://qcar_gazebo/meshes/QCarSteeringHubR.stl" scale="0.001 0.001 0.001"/>
+                <mesh filename="package://qcar_gazebo/models/qcar/QCarSteeringHubR.stl" scale="0.001 0.001 0.001"/>
             </geometry>
             <material name="orange"/>
@@ -96,5 +96,5 @@
             <origin rpy="0 0 0" xyz="0 0 0"/>
             <geometry>
-                <mesh filename="package://qcar_gazebo/meshes/QCarSteeringHubR.stl" scale="0.001 0.001 0.001"/>
+                <mesh filename="package://qcar_gazebo/models/qcar/QCarSteeringHubR.stl" scale="0.001 0.001 0.001"/>
             </geometry>
         </collision>
@@ -115,5 +115,5 @@
             <origin rpy="0 0 0" xyz="0 0 0"/>
             <geometry>
-                <mesh filename="package://qcar_gazebo/meshes/QCarWheel.stl" scale="0.001 0.001 0.001"/>
+                <mesh filename="package://qcar_gazebo/models/qcar/QCarWheel.stl" scale="0.001 0.001 0.001"/>
             </geometry>
             <material name="red"/>
@@ -122,5 +122,5 @@
             <origin rpy="0 0 0" xyz="0 0 0"/>
             <geometry>
-                <mesh filename="package://qcar_gazebo/meshes/QCarWheel.stl" scale="0.001 0.001 0.001"/>
+                <mesh filename="package://qcar_gazebo/models/qcar/QCarWheel.stl" scale="0.001 0.001 0.001"/>
             </geometry>
         </collision>
@@ -141,5 +141,5 @@
             <origin rpy="0 0 0" xyz="0 0 0"/>
             <geometry>
-                <mesh filename="package://qcar_gazebo/meshes/QCarWheel.stl" scale="0.001 0.001 0.001"/>
+                <mesh filename="package://qcar_gazebo/models/qcar/QCarWheel.stl" scale="0.001 0.001 0.001"/>
             </geometry>
             <material name="orange"/>
@@ -148,5 +148,5 @@
             <origin rpy="0 0 0" xyz="0 0 0"/>
             <geometry>
-                <mesh filename="package://qcar_gazebo/meshes/QCarWheel.stl" scale="0.001 0.001 0.001"/>
+                <mesh filename="package://qcar_gazebo/models/qcar/QCarWheel.stl" scale="0.001 0.001 0.001"/>
             </geometry>
         </collision>
@@ -167,5 +167,5 @@
             <origin rpy="0 0 0" xyz="0 0 0"/>
             <geometry>
-                <mesh filename="package://qcar_gazebo/meshes/QCarWheel.stl" scale="0.001 0.001 0.001"/>
+                <mesh filename="package://qcar_gazebo/models/qcar/QCarWheel.stl" scale="0.001 0.001 0.001"/>
             </geometry>
             <material name="orange"/>
@@ -174,5 +174,5 @@
             <origin rpy="0 0 0" xyz="0 0 0"/>
             <geometry>
-                <mesh filename="package://qcar_gazebo/meshes/QCarWheel.stl" scale="0.001 0.001 0.001"/>
+                <mesh filename="package://qcar_gazebo/models/qcar/QCarWheel.stl" scale="0.001 0.001 0.001"/>
             </geometry>
         </collision>
@@ -193,5 +193,5 @@
             <origin rpy="0 0 0" xyz="0 0 0"/>
             <geometry>
-                <mesh filename="package://qcar_gazebo/meshes/QCarWheel.stl" scale="0.001 0.001 0.001"/>
+                <mesh filename="package://qcar_gazebo/models/qcar/QCarWheel.stl" scale="0.001 0.001 0.001"/>
             </geometry>
             <material name="red"/>
@@ -200,5 +200,5 @@
             <origin rpy="0 0 0" xyz="0 0 0"/>
             <geometry>
-                <mesh filename="package://qcar_gazebo/meshes/QCarWheel.stl" scale="0.001 0.001 0.001"/>
+                <mesh filename="package://qcar_gazebo/models/qcar/QCarWheel.stl" scale="0.001 0.001 0.001"/>
             </geometry>
         </collision>
